File: bb-usb-buddy.sch (KiCad schematic (older format))
At the start: 2 parts, among them J1 USB_MICRO_B, J2 CONN_02X03

Commit message: guess i didnt need to invent my own micro usb connector.
Parts:
- removed J1: USB_MICRO_B, symbol USB_MICRO_B
- added J?: USB_OTG, Connectors:USB_Micro-B, symbol USB_OTG
- J2: footprint (none) -> Pin_Headers:Pin_Header_Straight_2x03_Pitch2.54mm
Connections:
- wire segments 17 -> 14
- no-connect marks 2 -> 3
Changed lines of the file:
@@
 LIBS:valves
 LIBS:usb_micro_b
+LIBS:bb-usb-buddy-cache
 EELAYER 25 0
 EELAYER END
@@
 $EndDescr
 $Comp
-L USB_MICRO_B J1
-U 1 1 596D8D41
-P 4000 3200
-F 0 "J1" H 3800 3650 50  0000 L CNN
-F 1 "USB_MICRO_B" H 3800 3550 50  0000 L CNN
-F 2 "" H 4150 3150 50  0001 C CNN
-F 3 "" H 4150 3150 50  0001 C CNN
-	1    4000 3200
+L GND #PWR02
+U 1 1 596D8E2E
+P 3950 3750
+F 0 "#PWR02" H 3950 3500 50  0001 C CNN
+F 1 "GND" H 3950 3600 50  0000 C CNN
+F 2 "" H 3950 3750 50  0001 C CNN
+F 3 "" H 3950 3750 50  0001 C CNN
+	1    3950 3750
 	1    0    0    -1
 $EndComp
 $Comp
-L GND #PWR01
-U 1 1 596D8E18
-P 3900 3700
-F 0 "#PWR01" H 3900 3450 50  0001 C CNN
-F 1 "GND" H 3900 3550 50  0000 C CNN
-F 2 "" H 3900 3700 50  0001 C CNN
-F 3 "" H 3900 3700 50  0001 C CNN
-	1    3900 3700
+L +5V #PWR03
+U 1 1 596D8ECB
+P 4250 2900
+F 0 "#PWR03" H 4250 2750 50  0001 C CNN
+F 1 "+5V" H 4250 3040 50  0000 C CNN
+F 2 "" H 4250 2900 50  0001 C CNN
+F 3 "" H 4250 2900 50  0001 C CNN
+	1    4250 2900
 	1    0    0    -1
 $EndComp
-$Comp
-L GND #PWR02
-U 1 1 596D8E2E
-P 4400 3500
-F 0 "#PWR02" H 4400 3250 50  0001 C CNN
-F 1 "GND" H 4400 3350 50  0000 C CNN
-F 2 "" H 4400 3500 50  0001 C CNN
-F 3 "" H 4400 3500 50  0001 C CNN
-	1    4400 3500
-	1    0    0    -1
-$EndComp
-Wire Wire Line
-	4300 3400 4400 3400
-Wire Wire Line
-	4400 3400 4400 3500
-Wire Wire Line
-	3900 3600 3900 3700
-NoConn ~ 4300 3200
-NoConn ~ 4300 3300
-$Comp
-L +5V #PWR03
-U 1 1 596D8ECB
-P 4400 3050
-F 0 "#PWR03" H 4400 2900 50  0001 C CNN
-F 1 "+5V" H 4400 3190 50  0000 C CNN
-F 2 "" H 4400 3050 50  0001 C CNN
-F 3 "" H 4400 3050 50  0001 C CNN
-	1    4400 3050
-	1    0    0    -1
-$EndComp
-Wire Wire Line
-	4400 3050 4400 3100
-Wire Wire Line
-	4400 3100 4300 3100
 $Comp
 L CONN_02X03 J2
@@
 F 0 "J2" H 5400 3450 50  0000 C CNN
 F 1 "CONN_02X03" H 5400 3050 50  0000 C CNN
-F 2 "" H 5400 2050 50  0001 C CNN
+F 2 "Pin_Headers:Pin_Header_Straight_2x03_Pitch2.54mm" H 5400 2050 50  0001 C CNN
 F 3 "" H 5400 2050 50  0001 C CNN
 	1    5400 3250
@@
 $EndComp
 Wire Wire Line
-	5100 2950 5100 3250
+	5100 2950 5100 3350
 Wire Wire Line
 	5100 3250 5150 3250
@@
 	5150 3150 5100 3150
 Connection ~ 5100 3150
+Connection ~ 5100 3000
+Wire Wire Line
+	5100 3350 5150 3350
+Connection ~ 5100 3250
 Wire Wire Line
 	5650 3150 5700 3150
 Wire Wire Line
-	5700 3150 5700 3000
-Wire Wire Line
-	5700 3000 5100 3000
-Connection ~ 5100 3000
+	5700 3150 5700 3550
 Wire Wire Line
 	5650 3250 5700 3250
-Wire Wire Line
-	5700 3250 5700 3550
+Connection ~ 5700 3250
 Wire Wire Line
 	5650 3350 5700 3350
 Connection ~ 5700 3350
+$Comp
+L USB_OTG J?
+U 1 1 596E9BEC
+P 3800 3200
+F 0 "J?" H 3600 3650 50  0000 L CNN
+F 1 "USB_OTG" H 3600 3550 50  0000 L CNN
+F 2 "Connectors:USB_Micro-B" H 3950 3150 50  0001 C CNN
+F 3 "" H 3950 3150 50  0001 C CNN
+	1    3800 3200
+	1    0    0    -1
+$EndComp
 Wire Wire Line
-	5150 3350 5100 3350
+	4100 3000 4250 3000
 Wire Wire Line
-	5100 3350 5100 3500
+	4250 3000 4250 2900
 Wire Wire Line
-	5100 3500 5700 3500
-Connection ~ 5700 3500
+	3700 3600 3700 3700
+Wire Wire Line
+	3700 3700 3950 3700
+Wire Wire Line
+	3800 3700 3800 3600
+Connection ~ 3800 3700
+Wire Wire Line
+	3950 3700 3950 3750
+NoConn ~ 4100 3200
+NoConn ~ 4100 3300
+NoConn ~ 4100 3400
 $EndSCHEMATC
